File: UU/kicad/uu_scheme/uu_scheme.kicad_sch (KiCad schematic)
At the start: 27 parts, among them J1 Screw_Terminal_01x03, J2 Conn_02x03_Odd_Even, SW1 SW_Push, U1 NRF24L01_Breakout, U2 PC817, U3 AMS1117-3.3, U4 STM32F103C6Tx

Commit message: УУ: незначательные изменения
Parts:
- renumbered C6 to C3, C3 to C5, C5 to C6, R5 to R3, R3 to R5, U2 to U1, U1 to U2
Changed lines of the file:
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@@
 		(on_board yes)
 		(dnp no)
-		(property "Reference" "U2"
+		(property "Reference" "U1"
 			(at 57.785 107.315 0)
 			(effects
@@
 			(project ""
 				(path "/07618df9-74d6-4e8c-8f50-1d30e388fe1d"
-					(reference "U2")
+					(reference "U1")
 					(unit 1)
 				)
@@
 		(dnp no)
 		(fields_autoplaced yes)
-		(property "Reference" "#PWR021"
+		(property "Reference" "#PWR014"
 			(at 126.365 140.335 0)
 			(effects
@@
 			(project ""
 				(path "/07618df9-74d6-4e8c-8f50-1d30e388fe1d"
-					(reference "#PWR021")
+					(reference "#PWR014")
 					(unit 1)
 				)
@@
 		(dnp no)
 		(fields_autoplaced yes)
-		(property "Reference" "#PWR017"
+		(property "Reference" "#PWR015"
 			(at 129.54 83.82 0)
 			(effects
@@
 			(project ""
 				(path "/07618df9-74d6-4e8c-8f50-1d30e388fe1d"
-					(reference "#PWR017")
+					(reference "#PWR015")
 					(unit 1)
 				)
@@
 		(on_board yes)
 		(dnp no)
-		(property "Reference" "R3"
+		(property "Reference" "R5"
 			(at 151.765 75.565 90)
 			(effects
@@
 			(project ""
 				(path "/07618df9-74d6-4e8c-8f50-1d30e388fe1d"
-					(reference "R3")
+					(reference "R5")
 					(unit 1)
 				)
@@
 		(dnp no)
 		(fields_autoplaced yes)
-		(property "Reference" "R5"
+		(property "Reference" "R3"
 			(at 144.78 118.11 90)
 			(effects
@@
 			(project ""
 				(path "/07618df9-74d6-4e8c-8f50-1d30e388fe1d"
-					(reference "R5")
+					(reference "R3")
 					(unit 1)
 				)
@@
 		(dnp no)
 		(fields_autoplaced yes)
-		(property "Reference" "#PWR01"
+		(property "Reference" "#PWR04"
 			(at 59.055 34.925 0)
 			(effects
@@
 			(project ""
 				(path "/07618df9-74d6-4e8c-8f50-1d30e388fe1d"
-					(reference "#PWR01")
+					(reference "#PWR04")
 					(unit 1)
 				)
@@
 		(dnp no)
 		(fields_autoplaced yes)
-		(property "Reference" "#PWR03"
+		(property "Reference" "#PWR07"
 			(at 76.835 22.86 0)
 			(effects
@@
 			(project ""
 				(path "/07618df9-74d6-4e8c-8f50-1d30e388fe1d"
-					(reference "#PWR03")
+					(reference "#PWR07")
 					(unit 1)
 				)
@@
 		(dnp no)
 		(fields_autoplaced yes)
-		(property "Reference" "#PWR016"
+		(property "Reference" "#PWR018"
 			(at 156.21 48.26 0)
 			(effects
@@
 			(project ""
 				(path "/07618df9-74d6-4e8c-8f50-1d30e388fe1d"
-					(reference "#PWR016")
+					(reference "#PWR018")
 					(unit 1)
 				)
@@
 		(dnp no)
 		(fields_autoplaced yes)
-		(property "Reference" "#PWR05"
+		(property "Reference" "#PWR010"
 			(at 84.455 39.37 0)
 			(effects
@@
 			(project ""
 				(path "/07618df9-74d6-4e8c-8f50-1d30e388fe1d"
-					(reference "#PWR05")
+					(reference "#PWR010")
 					(unit 1)
 				)
@@
 		(on_board yes)
 		(dnp no)
-		(property "Reference" "C3"
+		(property "Reference" "C5"
 			(at 142.24 32.385 0)
 			(effects
@@
 			(project "uu_scheme"
 				(path "/07618df9-74d6-4e8c-8f50-1d30e388fe1d"
-					(reference "C3")
+					(reference "C5")
 					(unit 1)
 				)
@@
 		(dnp no)
 		(fields_autoplaced yes)
-		(property "Reference" "#PWR04"
+		(property "Reference" "#PWR011"
 			(at 92.075 22.86 0)
 			(effects
@@
 			(project ""
 				(path "/07618df9-74d6-4e8c-8f50-1d30e388fe1d"
-					(reference "#PWR04")
+					(reference "#PWR011")
 					(unit 1)
 				)
@@
 		(dnp no)
 		(fields_autoplaced yes)
-		(property "Reference" "#PWR06"
+		(property "Reference" "#PWR05"
 			(at 65.405 102.235 0)
 			(effects
@@
 			(project ""
 				(path "/07618df9-74d6-4e8c-8f50-1d30e388fe1d"
-					(reference "#PWR06")
+					(reference "#PWR05")
 					(unit 1)
 				)
@@
 		(dnp no)
 		(fields_autoplaced yes)
-		(property "Reference" "#PWR014"
+		(property "Reference" "#PWR020"
 			(at 179.705 150.495 0)
 			(effects
@@
 			(project ""
 				(path "/07618df9-74d6-4e8c-8f50-1d30e388fe1d"
-					(reference "#PWR014")
+					(reference "#PWR020")
 					(unit 1)
 				)
@@
 		(dnp no)
 		(fields_autoplaced yes)
-		(property "Reference" "#PWR020"
+		(property "Reference" "#PWR013"
 			(at 126.365 130.81 0)
 			(effects
@@
 			(project ""
 				(path "/07618df9-74d6-4e8c-8f50-1d30e388fe1d"
-					(reference "#PWR020")
+					(reference "#PWR013")
 					(unit 1)
 				)
@@
 		(dnp no)
 		(fields_autoplaced yes)
-		(property "Reference" "#PWR02"
+		(property "Reference" "#PWR03"
 			(at 53.975 26.035 0)
 			(effects
@@
 			(project ""
 				(path "/07618df9-74d6-4e8c-8f50-1d30e388fe1d"
-					(reference "#PWR02")
+					(reference "#PWR03")
 					(unit 1)
 				)
@@
 		(dnp no)
 		(fields_autoplaced yes)
-		(property "Reference" "#PWR010"
+		(property "Reference" "#PWR01"
 			(at 31.75 71.12 0)
 			(effects
@@
 			(project "uu_scheme"
 				(path "/07618df9-74d6-4e8c-8f50-1d30e388fe1d"
-					(reference "#PWR010")
+					(reference "#PWR01")
 					(unit 1)
 				)
@@
 		(on_board yes)
 		(dnp no)
-		(property "Reference" "C5"
+		(property "Reference" "C6"
 			(at 153.035 32.385 0)
 			(effects
@@
 			(project ""
 				(path "/07618df9-74d6-4e8c-8f50-1d30e388fe1d"
-					(reference "C5")
+					(reference "C6")
 					(unit 1)
 				)
@@
 		(on_board yes)
 		(dnp no)
-		(property "Reference" "U1"
+		(property "Reference" "U2"
 			(at 84.455 63.4999 0)
 			(effects
@@
 			(project ""
 				(path "/07618df9-74d6-4e8c-8f50-1d30e388fe1d"
-					(reference "U1")
+					(reference "U2")
 					(unit 1)
 				)
@@
 		(dnp no)
 		(fields_autoplaced yes)
-		(property "Reference" "C6"
+		(property "Reference" "C3"
 			(at 133.35 72.3899 0)
 			(effects
@@
 			(project ""
 				(path "/07618df9-74d6-4e8c-8f50-1d30e388fe1d"
-					(reference "C6")
+					(reference "C3")
 					(unit 1)
 				)
@@
 		(dnp no)
 		(fields_autoplaced yes)
-		(property "Reference" "#PWR015"
+		(property "Reference" "#PWR017"
 			(at 156.21 30.48 0)
 			(effects
@@
 			(project ""
 				(path "/07618df9-74d6-4e8c-8f50-1d30e388fe1d"
-					(reference "#PWR015")
+					(reference "#PWR017")
 					(unit 1)
 				)
@@
 		(dnp no)
 		(fields_autoplaced yes)
-		(property "Reference" "#PWR07"
+		(property "Reference" "#PWR06"
 			(at 67.31 147.32 0)
 			(effects
@@
 			(project ""
 				(path "/07618df9-74d6-4e8c-8f50-1d30e388fe1d"
-					(reference "#PWR07")
+					(reference "#PWR06")
 					(unit 1)
 				)
@@
 		(dnp no)
 		(fields_autoplaced yes)
-		(property "Reference" "#PWR011"
+		(property "Reference" "#PWR02"
 			(at 40.64 77.47 0)
 			(effects
@@
 			(project ""
 				(path "/07618df9-74d6-4e8c-8f50-1d30e388fe1d"
-					(reference "#PWR011")
+					(reference "#PWR02")
 					(unit 1)
 				)
@@
 		(dnp no)
 		(fields_autoplaced yes)
-		(property "Reference" "#PWR013"
+		(property "Reference" "#PWR019"
 			(at 178.435 60.96 0)
 			(effects
@@
 			(project ""
 				(path "/07618df9-74d6-4e8c-8f50-1d30e388fe1d"
-					(reference "#PWR013")
+					(reference "#PWR019")
 					(unit 1)
 				)
@@
 		(dnp no)
 		(fields_autoplaced yes)
-		(property "Reference" "#PWR019"
+		(property "Reference" "#PWR016"
 			(at 145.415 79.375 0)
 			(effects
@@
 			(project ""
 				(path "/07618df9-74d6-4e8c-8f50-1d30e388fe1d"
-					(reference "#PWR019")
+					(reference "#PWR016")
 					(unit 1)
 				)
@@
 		(dnp no)
 		(fields_autoplaced yes)
-		(property "Reference" "#PWR018"
+		(property "Reference" "#PWR012"
 			(at 114.935 76.2 0)
 			(effects
@@
 			(project ""
 				(path "/07618df9-74d6-4e8c-8f50-1d30e388fe1d"
-					(reference "#PWR018")
+					(reference "#PWR012")
 					(unit 1)
 				)
